File: mcm_r/mcm_r_kicad/mcm_r_kicad.kicad_sch (KiCad schematic)
At the start: 34 parts, among them U1 RP2350_60QFN, U2 W25Q32JVSS, U3 APS6404L-3SQN

Commit message: 20241214-1 update readme and swap MCM R's battery chip
Parts:
- removed L?: L_Small, symbol Device:L_Small
- removed R?: 550K, symbol Device:R_Small
- removed R?: 145K, symbol Device:R_Small
- removed SW?: SW_Push, symbol Switch:SW_Push
- removed U?: LTC3553, Package_DFN_QFN:QFN-20-1EP_3x3mm_P0.4mm_EP1.65x1.65mm, symbol Battery_Management:LTC3553
Other:
- note added: "October 20, 2024 - December 14, 2024"
- note removed: "October 20, 2024 - November 6, 2024"
- moved on the sheet: C?
